File: schematic/schematic.kicad_sch (KiCad schematic)
At the start: 28 parts, among them M1 Motor_DC, M2 Motor_DC, M3 Motor_Servo, M4 Motor_DC, M5 Motor_DC

Commit message: Switched to tank drive
Parts:
- removed C5: 470uf, Package_DFN_QFN:WDFN-10-1EP_3x3mm_P0.5mm_EP1.8x2.5mm, symbol Device:C_Polarized_US
- removed C7: 0.1uf, symbol Device:C
- removed M3: Motor_Servo, symbol Motor:Motor_Servo
Connections:
- net GPIO23: now also U2.1 (R_PWM)
- net GPIO3: now reaches U3.27 (GPIO3)
- net GPIO3: now also U2.4 (L_EN)
- net GPIO1: now reaches U3.28 (GPIO1)
- net GPIO1: now also U2.3 (R_EN)
- net GPIO22: now reaches U3.29 (GPIO22)
- net GPIO22: now also U2.2 (L_PWM)
- net GPIO12: no longer names the net of U3.4 (GPIO12)
- net GPIO12: no longer U2.3 (R_EN)
- net GPIO13: no longer names the net of U3.3 (GPIO13)
- net GPIO13: no longer U2.4 (L_EN)
- net GPIO14: no longer names the net of U3.5 (GPIO14)
- net GPIO14: no longer U2.2 (L_PWM)
- net GPIO27: no longer names the net of U3.6 (GPIO27)
- net GPIO27: no longer U2.1 (R_PWM)
- no-connect marks 22 -> 23
Other:
- note added: "(Input Only)"
- moved on the sheet: BT1, C1, C10, C11, C12, C13, C14, C15, C16, C17, C18, C2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
